Commit message: added main wheels and castor wheel to bot

File: mechbot_description/urdf/bot.urdf (robot description, URDF)
Before this commit: robot bot, 2 links, 1 joints
Links:
- added link front_castor_link; visual sphere radius=0.0075
- added link left_wheel_link; visual cylinder length=0.02 radius=0.04
- added link rear_castor_link; visual sphere radius=0.0075
- added link right_wheel_link; visual cylinder length=0.02 radius=0.04
Joints:
- added joint front_castor_joint: type fixed, parent base_link, child front_castor_link, origin xyz=0.0 0.07 -0.0315 rpy=0.0 1.57 0.0
- added joint left_wheel_joint: type fixed, parent base_link, child left_wheel_link, origin xyz=-0.06 0.0 0.0 rpy=0.0 1.57 0.0
- added joint rear_castor_joint: type fixed, parent base_link, child rear_castor_link, origin xyz=0.0 -0.07 -0.0315 rpy=0.0 1.57 0.0
- added joint right_wheel_joint: type fixed, parent base_link, child right_wheel_link, origin xyz=0.06 0.0 0.0 rpy=0.0 1.57 0.0
- joint base_joint: origin xyz=0.0 0.0 0.15 rpy=0.0 0.0 0.0 -> xyz=0.0 0.0 0.04 rpy=0.0 0.0 1.57
